Commit message: updated robot

File: robot/panda.urdf.xacro (robot description, xacro)
@@ -2,5 +2,5 @@
 <robot xmlns:xacro="http://www.ros.org/wiki/xacro" name="panda">
     <xacro:arg name="robot_name" default="panda"/>
-    <xacro:include filename="$(find joint_velocity_controller)/robot/panda.xacro" />
+    <xacro:include filename="$(find dynamics_wrapper)/robot/panda.xacro" />
     <xacro:panda_arm robot_name="$(arg robot_name)"/>
 </robot>

File: robot/panda.xacro (robot description, xacro)
@@ -1,5 +1,5 @@
 <?xml version='1.0' encoding='utf-8'?>
 <robot xmlns:xacro="http://www.ros.org/wiki/xacro" name="panda">
-    <xacro:macro name="panda_arm" params="robot_name description_pkg:='franka_description' ">
+    <xacro:macro name="panda_arm" params="robot_name ">
         <link name = "world"/>
         <link name="${robot_name}_link0">
